File: TimeCapsulePCB/TimeCapsule.kicad_sch (KiCad schematic)
At the start: 53 parts, among them J1 USB_C_Receptacle_USB2.0_14P, Q1 Q_PMOS_GSD, Q2 Q_NMOS_GSD, Q3 Q_NMOS_GSD, Q4 Q_NMOS_GSD, SW1 SW_Push, SW2 SW_Push, U1 RP2040, U2 TPL5110, U3 AP2112K-3.3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

Commit message: Update readme and BOM
Parts:
- R11: DIGIKEY # YAG3003CT-ND -> P16.9KLCT-ND; MANUFACTURER YAGEO -> Panasonic Electronic Components; MPN RC0402FR-0716K9L -> ERJ-2RKF1692X
- R3, R4: DIGIKEY # YAG3085CT-ND -> 738-RMCF0402FT27R4CT-ND; MANUFACTURER YAGEO -> Stackpole Electronics Inc; MPN RC0402FR-0727R4L -> RMCF0402FT27R4
Changed lines of the file:
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@@
 			)
 		)
-		(property "DIGIKEY #" "YAG3003CT-ND"
+		(property "DIGIKEY #" "P16.9KLCT-ND"
 			(at 53.34 238.76 90)
 			(effects
@@
 			)
 		)
-		(property "MPN" "RC0402FR-0716K9L"
+		(property "MPN" "ERJ-2RKF1692X"
 			(at 53.34 238.76 90)
 			(effects
@@
 			)
 		)
-		(property "MANUFACTURER" "YAGEO"
+		(property "MANUFACTURER" "Panasonic Electronic Components"
 			(at 53.34 238.76 90)
 			(effects
@@
 			)
 		)
-		(property "DIGIKEY #" "YAG3085CT-ND"
+		(property "DIGIKEY #" "738-RMCF0402FT27R4CT-ND"
 			(at 35.56 67.31 90)
 			(effects
@@
 			)
 		)
-		(property "MPN" "RC0402FR-0727R4L"
+		(property "MPN" "RMCF0402FT27R4"
 			(at 35.56 67.31 90)
 			(effects
@@
 			)
 		)
-		(property "MANUFACTURER" "YAGEO"
+		(property "MANUFACTURER" "Stackpole Electronics Inc"
 			(at 35.56 67.31 90)
 			(effects
@@
 			)
 		)
-		(property "DIGIKEY #" "YAG3085CT-ND"
+		(property "DIGIKEY #" "738-RMCF0402FT27R4CT-ND"
 			(at 35.56 76.2 90)
 			(effects
@@
 			)
 		)
-		(property "MPN" "RC0402FR-0727R4L"
+		(property "MPN" "RMCF0402FT27R4"
 			(at 35.56 76.2 90)
 			(effects
@@
 			)
 		)
-		(property "MANUFACTURER" "YAGEO"
+		(property "MANUFACTURER" "Stackpole Electronics Inc"
 			(at 35.56 76.2 90)
 			(effects
